Commit message: camera_rotation_fixed

File: src/my_robot/urdf/my_robot.xacro (robot description, xacro)
@@ -187,5 +187,5 @@
         </joint>
 	  <joint name="camera_optical_joint" type="fixed">
-    <origin xyz="0 0 0" rpy="-1.5707 0 -1.5707"/>
+    <origin xyz="0 0 0" rpy="0 0 0"/>
     <parent link="camera"/>
     <child link="camera_link_optical"/>

Commit message: 06-07-21

File: src/my_robot/urdf/my_robot.xacro (robot description, xacro)
@@ -187,5 +187,5 @@
         </joint>
 	  <joint name="camera_optical_joint" type="fixed">
-    <origin xyz="0 0 0" rpy="0 0 0"/>
+    <origin xyz="0 0 0" rpy="-1.5707 0 -1.5707"/>
     <parent link="camera"/>
     <child link="camera_link_optical"/>
